File: HVI design.kicad_sch (KiCad schematic)
At the start: 24 parts, among them Q1 TK3P80E, U1 LT8316EFE, U2 TLV1702

Commit message: Add files via upload
Parts:
- removed U2: TLV1702, Custom_MSM:Comparator_Dual_VSSOP-8, symbol Custom_MSM:Comparator_Dual_Open-Coll
- added D4: LED, symbol Device:LED
- added F1: Fuse, symbol Device:Fuse
- added J1: HV+, Custom_MSM:Connector_PP15, symbol Custom_MSM:Connector_PP15
- added J2: HV-, Custom_MSM:Connector_PP15, symbol Custom_MSM:Connector_PP15
- added R2: R, symbol Device:R
- added U3: PEME1-S12-S5-S, Converter_DCDC:Converter_DCDC_Murata_CRE1xxxxxxSC_THT, symbol Regulator_Switching:CRE1S1205SC
Connections:
- net GND: now also J2.1 (Pin_1), J2.2 (Pin_2), U3.2 (GND)
- net at C6.1, C7.1, C8.1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: now also U3.1 (+VIN)
- net V_In renamed E1
- net E1: now also F1.2
- new net: F1.1, J1.1 (Pin_1), J1.2 (Pin_2)
- new net: D4.2 (A), R2.1
- new net: R2.2, U3.7 (+VOUT)
- new net: D4.1 (K), U3.5 (0V)
Other:
- note added: "(soon to be high voltage indicator LCD screen)"
- note added: "12V 10-200mA"
- note added: "Demonstration circuit 2781A is a nonisolated buck converter featuring the LT8316. The demo board outputs 12V and maintains tight regulation with a load current from 10mA to 0.2A. It is optimized to operate over a wide 19V to 600V DC input voltage range. Output voltage accuracy stays within ±1% over the entire input voltage and load range."
- note added: "High Voltage Indicator Light"
- note added: "Vin+"
- note added: "Vin-"
- note added: "Vout+"
- note added: "Vout-"
- note added: "isolated DC-DC converter 5V <- (10.8 - 13.2V)"
- title: (none) -> High Voltage Indicator Light FS2026 EV
- moved on the sheet: C1, C10, C2, C3, C4, C5, C6, C7, C8, D1, D2, D3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

Commit message: Add files via upload
Parts:
- removed U3: PEME1-S12-S5-S, Converter_DCDC:Converter_DCDC_Murata_CRE1xxxxxxSC_THT, symbol Regulator_Switching:CRE1S1205SC
- added J1: HV+, Custom_MSM:Connector_PP15, symbol Custom_MSM:Connector_PP15
- added J2: HV-, Custom_MSM:Connector_PP15, symbol Custom_MSM:Connector_PP15
- added R10: 30k, symbol Device:R
- added R11: 10k, symbol Device:R
- added R5, R7: 600k, symbol Device:R
- added R6: 700k, symbol Device:R
- added R8, R9: 100k, symbol Device:R
- added U2: TLV1702, Custom_MSM:Comparator_Dual_VSSOP-8, symbol Custom_MSM:Comparator_Dual_Open-Coll
- R2: value R -> 10k
Connections:
- net GND: now also D4.1 (K), R11.1
- net at C6.1, C7.1, C8.1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: now also R10.1, R9.1
- net at R2.2: now also R9.2, U2.1
- new net: R6.2, R7.1
- new net: R10.2, R11.2, U2.3 (+)
- new net: J2.1 (Pin_1), J2.2 (Pin_2), R8.2
- new net: R5.2, R6.1
- new net: U1.2 (VIN), U1.3 (VIN) (x2)
- new net: J1.1 (Pin_1), J1.2 (Pin_2), R5.1
- new net 1/20_V_divider: R7.2, R8.1, U2.2 (-)
Other:
- note added: "Voltage divider to take 1/5 of the V from TSAC"
- note added: "output = high when TSAC voltage is 60V, as the 1/20 scaled TSAC voltage is compared to a 12V voltage from the eval board output."
- note removed: "isolated DC-DC converter 5V <- (10.8 - 13.2V)"
- moved on the sheet: F1, J1, J2

Commit message: Add files via upload
Parts:
- removed JP1: Jumper_3_Bridged12, symbol Jumper:Jumper_3_Bridged12
- J3: renamed from J1; value HV+ -> V+
- J4: renamed from J2; value HV- -> V-
- R10: value 30k -> 31.6k
Connections:
- net 1/20_V_divider: now also U2.3 (+); no longer U2.2 (-)
- net GND: no longer U1.16 (SMODE)
- net INTVcc: now also U1.16 (SMODE)
- net 2.88V_reference: now reaches R10.2, R11.2
- net 2.88V_reference: now also U2.2 (-); no longer U2.3 (+)
- new net: U1.2 (VIN), U1.3 (VIN) (x2)
Other:
- note added: "3V when V=60V"
- note added: "A 2.88V reference voltage is used to compensate for the fact that the DC2718 can output 11.6-12.4V, so when the DC2718A outputs 12V the V threshold for comparator output becomes 57.6V."
- note added: "V is scaled by 1/20 as the TV comparator has a maximum voltage rating of 36V, so using this divider the max input (450V detected) will be ~22.5V, and at 60V measured voltage the output will be 3V."
- note added: "Voltage divider to take 1/20 of the V from vehicle side of AIR's"
- note added: "output = high when measured voltage is 57.6V, as the 1/20 scaled voltage is compared to the 12V output from the eval board."
- note added: "~450V max"
- note removed: "Voltage divider to take 1/5 of the V from TSAC"
- note removed: "output = high when TSAC voltage is 60V, as the 1/20 scaled TSAC voltage is compared to a 12V voltage from the eval board output."
Changed lines of the file:
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@@
 		)
 	)
-	(text "output = high when TSAC voltage is 60V, as the \n1/20 scaled TSAC voltage is compared to a \n12V voltage from the eval board\noutput."
+	(text "output = high when measured voltage \nis 57.6V, as the 1/20 scaled voltage \nis compared to the 12V output from \nthe eval board.\n"
 		(exclude_from_sim no)
-		(at 288.544 203.2 0)
+		(at 288.544 217.17 0)
 		(effects
 			(font
@@
 		)
 	)
+	(text "V is scaled by 1/20 as the TV comparator \nhas a maximum voltage rating of 36V, so \nusing this divider the max input (450V detected) \nwill be ~22.5V, and at 60V measured voltage the \noutput will be 3V."
+		(exclude_from_sim no)
+		(at 99.822 244.856 0)
+		(effects
+			(font
+				(size 1.27 1.27)
+			)
+		)
+	)
 	(text "(soon to be high voltage indicator LCD screen)"
 		(exclude_from_sim no)
@@
 		)
 	)
+	(text "~450V max\n"
+		(exclude_from_sim no)
+		(at 101.092 99.314 0)
+		(effects
+			(font
+				(size 1.27 1.27)
+			)
+		)
+	)
 	(text "Demonstration circuit 2781A is a nonisolated buck converter \nfeaturing the LT8316. The demo board outputs 12V and maintains \ntight regulation with a load current from 10mA to 0.2A. It is \noptimized to operate over a wide 19V to 600V DC input voltage \nrange. Output voltage accuracy stays within ±1% over the entire \ninput voltage and load range."
 		(exclude_from_sim no)
@@
 		)
 	)
+	(text "A 2.88V reference voltage is used to \ncompensate for the fact that the DC2718 \ncan output 11.6-12.4V, so when the DC2718A \noutputs 12V the V threshold for comparator \noutput becomes 57.6V."
+		(exclude_from_sim no)
+		(at 366.776 200.66 0)
+		(effects
+			(font
+				(size 1.27 1.27)
+			)
+		)
+	)
 	(text "12V \n10-200mA"
 		(exclude_from_sim no)
@@
 		)
 	)
+	(text "3V when V=60V"
+		(exclude_from_sim no)
+		(at 308.864 187.198 0)
+		(effects
+			(font
+				(size 1.27 1.27)
+			)
+		)
+	)
 	(text "Vin-"
 		(exclude_from_sim no)
@@
 		)
 	)
-	(text "Voltage divider to take 1/5 of the V from TSAC"
+	(text "Voltage divider to take 1/20 of the V from vehicle side of AIR's"
 		(exclude_from_sim no)
 		(at 45.466 220.472 0)
@@
 	)
 	(junction
-		(at 331.47 187.96)
-		(diameter 0)
-		(color 0 0 0 0)
-	)
-	(junction
 		(at 38.1 267.97)
 		(diameter 0)
@@
 	)
 	(junction
-		(at 213.36 143.51)
-		(diameter 0)
-		(color 0 0 0 0)
-	)
-	(junction
 		(at 284.48 190.5)
 		(diameter 0)
@@
 	)
 	(junction
-		(at 228.6 143.51)
-		(diameter 0)
-		(color 0 0 0 0)
-	)
-	(junction
 		(at 237.49 143.51)
 		(diameter 0)
@@
 	)
 	(junction
+		(at 331.47 193.04)
+		(diameter 0)
+		(color 0 0 0 0)
+	)
+	(junction
 		(at 38.1 232.41)
 		(diameter 0)
@@
 	(wire
 		(pts
-			(xy 358.14 193.04) (xy 299.72 193.04)
-		)
-		(stroke
-			(width 0)
-			(type default)
-		)
-	)
-	(wire
-		(pts
 			(xy 237.49 143.51) (xy 250.19 143.51)
 		)
@@
 	(wire
 		(pts
-			(xy 228.6 143.51) (xy 220.98 143.51)
+			(xy 299.72 193.04) (xy 331.47 193.04)
+		)
+		(stroke
+			(width 0)
+			(type default)
+		)
+	)
+	(wire
+		(pts
+			(xy 220.98 143.51) (xy 237.49 143.51)
 		)
 		(stroke
@@
 	(wire
 		(pts
-			(xy 87.63 90.17) (xy 87.63 91.44)
+			(xy 331.47 193.04) (xy 331.47 196.85)
 		)
 		(stroke
@@
 	(wire
 		(pts
-			(xy 250.19 90.17) (xy 270.51 90.17)
+			(xy 87.63 90.17) (xy 87.63 91.44)
 		)
 		(stroke
@@
 	(wire
 		(pts
-			(xy 331.47 187.96) (xy 331.47 196.85)
+			(xy 250.19 90.17) (xy 270.51 90.17)
 		)
 		(stroke
@@
 	(wire
 		(pts
-			(xy 199.39 128.27) (xy 199.39 127)
+			(xy 213.36 127) (xy 213.36 129.54)
 		)
 		(stroke
@@
 	(wire
 		(pts
-			(xy 318.77 152.4) (xy 318.77 153.67)
-		)
-		(stroke
-			(width 0)
-			(type default)
-		)
-	)
-	(wire
-		(pts
-			(xy 256.54 143.51) (xy 250.19 143.51)
+			(xy 199.39 128.27) (xy 199.39 127)
 		)
 		(stroke
@@
 	(wire
 		(pts
-			(xy 220.98 143.51) (xy 213.36 143.51)
+			(xy 318.77 152.4) (xy 318.77 153.67)
 		)
 		(stroke
@@
 	(wire
 		(pts
-			(xy 228.6 153.67) (xy 228.6 143.51)
+			(xy 256.54 143.51) (xy 250.19 143.51)
 		)
 		(stroke
@@
 	(wire
 		(pts
-			(xy 299.72 187.96) (xy 331.47 187.96)
-		)
-		(stroke
-			(width 0)
-			(type default)
-		)
-	)
-	(wire
-		(pts
 			(xy 87.63 106.68) (xy 87.63 107.95)
 		)
@@
 	(wire
 		(pts
-			(xy 199.39 143.51) (xy 213.36 143.51)
+			(xy 199.39 143.51) (xy 220.98 143.51)
 		)
 		(stroke
@@
 	(wire
 		(pts
-			(xy 219.71 153.67) (xy 228.6 153.67)
-		)
-		(stroke
-			(width 0)
-			(type default)
-		)
-	)
-	(wire
-		(pts
-			(xy 201.93 153.67) (xy 207.01 153.67)
-		)
-		(stroke
-			(width 0)
-			(type default)
-		)
-	)
-	(wire
-		(pts
 			(xy 250.19 143.51) (xy 250.19 113.03)
 		)
@@
 	(wire
 		(pts
-			(xy 213.36 143.51) (xy 213.36 149.86)
-		)
-		(stroke
-			(width 0)
-			(type default)
-		)
-	)
-	(wire
-		(pts
 			(xy 220.98 137.16) (xy 220.98 143.51)
 		)
@@
 	(wire
 		(pts
-			(xy 213.36 127) (xy 213.36 143.51)
-		)
-		(stroke
-			(width 0)
-			(type default)
-		)
-	)
-	(wire
-		(pts
 			(xy 250.19 113.03) (xy 256.54 113.03)
 		)
@@
 	(wire
 		(pts
-			(xy 228.6 143.51) (xy 237.49 143.51)
-		)
-		(stroke
-			(width 0)
-			(type default)
-		)
-	)
-	(wire
-		(pts
 			(xy 154.94 118.11) (xy 154.94 114.3)
 		)
@@
 	(wire
 		(pts
-			(xy 331.47 184.15) (xy 331.47 187.96)
+			(xy 331.47 184.15) (xy 331.47 193.04)
+		)
+		(stroke
+			(width 0)
+			(type default)
+		)
+	)
+	(wire
+		(pts
+			(xy 299.72 187.96) (xy 339.09 187.96)
 		)
 		(stroke
@@
 		)
 	)
+	(label "2.88V_reference"
+		(at 302.26 193.04 0)
+		(effects
+			(font
+				(size 1.27 1.27)
+			)
+			(justify left bottom)
+		)
+	)
 	(global_label "1/20_V_divider"
 		(shape input)
-		(at 358.14 193.04 0)
+		(at 339.09 187.96 0)
 		(fields_autoplaced yes)
 		(effects
@@
 		)
 		(property "Intersheetrefs" "${INTERSHEET_REFS}"
-			(at 374.2485 193.04 0)
+			(at 355.1985 187.96 0)
 			(effects
 				(font
@@
 	(global_label "INTVcc"
 		(shape input)
-		(at 201.93 153.67 180)
+		(at 213.36 129.54 270)
 		(fields_autoplaced yes)
 		(effects
@@
 		)
 		(property "Intersheetrefs" "${INTERSHEET_REFS}"
-			(at 192.7761 153.67 0)
+			(at 213.36 138.6939 90)
 			(effects
 				(font
@@
 	)
 	(symbol
-		(lib_id "Jumper:Jumper_3_Bridged12")
-		(at 213.36 153.67 180)
-		(unit 1)
-		(exclude_from_sim no)
-		(in_bom no)
-		(on_board yes)
-		(dnp no)
-		(fields_autoplaced yes)
-		(property "Reference" "JP1"
-			(at 213.36 157.48 0)
-			(effects
-				(font
-					(size 1.27 1.27)
-				)
-			)
-		)
-		(property "Value" "Jumper_3_Bridged12"
-			(at 213.36 160.02 0)
-			(effects
-				(font
-					(size 1.27 1.27)
-				)
-			)
-		)
-		(property "Footprint" ""
-			(at 213.36 153.67 0)
-			(effects
-				(font
-					(size 1.27 1.27)
-				)
-				(hide yes)
-			)
-		)
-		(property "Datasheet" "~"
-			(at 213.36 153.67 0)
-			(effects
-				(font
-					(size 1.27 1.27)
-				)
-				(hide yes)
-			)
-		)
-		(property "Description" "Jumper, 3-pole, pins 1+2 closed/bridged"
-			(at 213.36 153.67 0)
-			(effects
-				(font
-					(size 1.27 1.27)
-				)
-				(hide yes)
-			)
-		)
-		(pin "2"
-		)
-		(pin "1"
-		)
-		(pin "3"
-		)
-		(instances
-			(project ""
-				(path "/6e774aff-27e0-4346-9be8-67b840f3c91a"
-					(reference "JP1")
-					(unit 1)
-				)
-			)
-		)
-	)
-	(symbol
 		(lib_id "Device:L")
 		(at 270.51 143.51 90)
@@
 			)
 		)
-		(property "Value" "30k"
+		(property "Value" "31.6k"
 			(at 334.01 181.6099 0)
 			(effects
@@
 		(on_board yes)
 		(dnp no)
-		(property "Reference" "J2"
-			(at 44.831 276.733 90)
+		(property "Reference" "J4"
+			(at 42.926 276.606 90)
 			(effects
 				(font
@@
 			)
 		)
-		(property "Value" "HV-"
-			(at 44.831 274.193 90)
+		(property "Value" "V-"
+			(at 42.926 274.066 90)
 			(effects
 				(font
@@
 			(project "HVI design"
 				(path "/6e774aff-27e0-4346-9be8-67b840f3c91a"
-					(reference "J2")
+					(reference "J4")
 					(unit 1)
 				)
@@
 		(on_board yes)
 		(dnp no)
-		(fields_autoplaced yes)
-		(property "Reference" "J1"
-			(at 41.91 224.7899 90)
+		(property "Reference" "J3"
+			(at 41.91 225.044 90)
 			(effects
 				(font
@@
 			)
 		)
-		(property "Value" "HV+"
-			(at 41.91 227.3299 90)
+		(property "Value" "V+"
+			(at 41.91 227.584 90)
 			(effects
 				(font
@@
 			(project "HVI design"
 				(path "/6e774aff-27e0-4346-9be8-67b840f3c91a"
-					(reference "J1")
+					(reference "J3")
 					(unit 1)
 				)

Commit message: Add files via upload
Parts:
- C10: value 0.1 µF -> 0.1µF
- C2: value optional -> 10nF
- C4: value C -> 10uF
- R1: value R -> 2.49k
- R3: value R -> 21.5k
Connections:
- new net: U1.2 (VIN), U1.3 (VIN) (x2)
Other:
- moved on the sheet: F1
Changed lines of the file:
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@@
 	(wire
 		(pts
-			(xy 101.6 91.44) (xy 119.38 91.44)
+			(xy 99.06 91.44) (xy 119.38 91.44)
 		)
 		(stroke
@@
 	(wire
 		(pts
-			(xy 87.63 91.44) (xy 93.98 91.44)
+			(xy 87.63 91.44) (xy 91.44 91.44)
 		)
 		(stroke
@@
 		(dnp no)
 		(property "Reference" "C2"
-			(at 114.3 97.028 0)
+			(at 113.538 97.282 0)
 			(effects
 				(font
@@
 			)
 		)
-		(property "Value" "optional"
-			(at 109.22 99.822 0)
+		(property "Value" "10nF"
+			(at 112.522 99.314 0)
 			(effects
 				(font
@@
 	(symbol
 		(lib_id "Device:Fuse")
-		(at 97.79 91.44 90)
+		(at 95.25 91.44 90)
 		(unit 1)
 		(exclude_from_sim no)
@@
 		(fields_autoplaced yes)
 		(property "Reference" "F1"
-			(at 97.79 85.09 90)
+			(at 95.25 85.09 90)
 			(effects
 				(font
@@
 		)
 		(property "Value" "Fuse"
-			(at 97.79 87.63 90)
+			(at 95.25 87.63 90)
 			(effects
 				(font
@@
 		)
 		(property "Footprint" ""
-			(at 97.79 93.218 90)
+			(at 95.25 93.218 90)
 			(effects
 				(font
@@
 		)
 		(property "Datasheet" "~"
-			(at 97.79 91.44 0)
+			(at 95.25 91.44 0)
 			(effects
 				(font
@@
 		)
 		(property "Description" "Fuse"
-			(at 97.79 91.44 0)
+			(at 95.25 91.44 0)
 			(effects
 				(font
@@
 			)
 		)
-		(property "Value" "0.1 µF"
-			(at 201.93 133.35 0)
+		(property "Value" "0.1µF"
+			(at 201.93 132.842 0)
 			(effects
 				(font
@@
 		(dnp no)
 		(property "Reference" "R4"
-			(at 188.976 131.318 0)
+			(at 187.706 131.318 0)
 			(effects
 				(font
@@
 		)
 		(property "Value" "22.1k"
-			(at 186.69 133.35 0)
+			(at 186.182 133.35 0)
 			(effects
 				(font
@@
 		(dnp no)
 		(property "Reference" "R3"
-			(at 260.858 110.998 0)
+			(at 262.636 108.966 90)
 			(effects
 				(font
@@
 			)
 		)
-		(property "Value" "R"
-			(at 262.8899 110.49 0)
+		(property "Value" "21.5k"
+			(at 264.414 110.744 90)
 			(effects
 				(font
@@
 			)
 		)
-		(property "Value" "R"
+		(property "Value" "2.49k"
 			(at 259.08 129.5399 0)
 			(effects
@@
 		(dnp no)
 		(property "Reference" "C5"
-			(at 196.596 137.922 0)
+			(at 186.182 138.43 0)
 			(effects
 				(font
@@
 		)
 		(property "Value" "0.1µF"
-			(at 195.58 139.7 0)
+			(at 185.166 140.208 0)
 			(effects
 				(font
@@
 		(on_board yes)
 		(dnp no)
-		(fields_autoplaced yes)
 		(property "Reference" "C4"
 			(at 254 96.5199 0)
@@
 			)
 		)
-		(property "Value" "C"
-			(at 254 99.0599 0)
+		(property "Value" "10uF"
+			(at 253.238 98.298 0)
 			(effects
 				(font

Commit message: Add files via upload
Parts:
- removed R11: 10k, symbol Device:R
- added Q2: BSS205N, Custom_MSM:MOSFET_Single_SOT-23, symbol Custom_MSM:MOSFET_N-CH
- added R12, R14: 10k, symbol Device:R
- added R13: 31.6k, symbol Device:R
- added U3: PC817, Package_DIP:DIP-4_W7.62mm, symbol Isolator:PC817
- R10: value 31.6k -> 1MΩ
- R9: value 100k -> 390Ω
Connections:
- net 1/20_V_divider: now also R10.2
- net 2.88V_reference: now also R13.2, R14.2; no longer R10.2
- net GND: now also R2.2, R9.1, Q2.3 (D), R12.1, R13.1; no longer D4.1 (K)
- net V-(12V): now reaches C6.1, C7.1, C8.1, D1.1 (K), D3.2 (A), L1.2
- net V-(12V): now also R14.1; no longer R10.1, R9.1
- net at R2.1: now also R10.1, U2.1, Q2.1 (G); no longer D4.2 (A)
- new net: D4.1 (K), U3.3
- new net: D4.2 (A), R12.2, U3.4
- new net: R9.2, U3.1
- new net: Q2.2 (S), U3.2
- new net: U1.2 (VIN), U1.3 (VIN) (x2)
Other:
- note added: "2.88V voltage reference from buck converter 12V output"
- note added: "N-channel MOSFET to drive the output voltage HIGH"
- note added: "hysteresis resistor"
- note added: "output = low when measured voltage is 57.6V (as TVL1702 is open-drain), as the 1/20 scaled voltage is compared to the 12V output from the eval board."
- note removed: "output = high when measured voltage is 57.6V, as the 1/20 scaled voltage is compared to the 12V output from the eval board."
- moved on the sheet: C1, C10, C2, C3, C4, C5, C6, C7, C8, D1, D2, D3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
